Commit message: Added modified gazebo_cave_world to the main repository

File: install/tello_description/share/tello_description/urdf/tello.urdf.xacro (robot description, xacro)
@@ -2,5 +2,5 @@
 <!-- Body coordinates are: x forward, y left, z up; rotation is: roll right, pitch forward, yaw left -->
 <!-- See http://www.ros.org/reps/rep-0103.html -->
-<robot name="tello">
+<robot name="tello" xmlns:xacro="http://ros.org/wiki/xacro">
     <!-- Materials -->
     <material name="gray">
@@ -174,4 +174,95 @@
         <axis xyz="0 0 1"/>
     </joint>
+    <link name="camera_optical_frame"/>
+    <joint name="camera_joint" type="fixed">
+        <origin xyz="0.059 0 0" rpy="0 0 0"/>
+        <parent link="base_link"/>
+        <child link="camera_optical_frame"/>
+    </joint>
+    <gazebo reference="camera_optical_frame">
+        <sensor name="depth_camera" type="depth">
+            <update_rate>10</update_rate>
+            <topic>ircam1</topic>
+            <camera>
+            <horizontal_fov>1.05</horizontal_fov>
+            <image>
+                <width>640</width>
+                <height>480</height>
+                <format>R_FLOAT32</format>
+            </image>
+            <clip>
+                <near>0.1</near>
+                <far>10.0</far>
+            </clip>
+            </camera>
+            <always_on>true</always_on>
+            <visualize>true</visualize>
+        </sensor>
+    </gazebo>
+    <gazebo reference="base_link">
+        <sensor name="imu_sensor" type="imu">
+        <topic>/tello/imu</topic>
+        <plugin filename="gz-sim-imu-system" name="gz::sim::systems::Imu">
+            <initial_orientation_as_reference>false</initial_orientation_as_reference>
+        </plugin>
+        <always_on>true</always_on>
+        <update_rate>200</update_rate>
+        <visualize>true</visualize>
+        <imu>
+            <angular_velocity>
+            <x>
+                <noise type="gaussian">
+                <mean>0.0</mean>
+                <stddev>2e-4</stddev>
+                <bias_mean>0.0000075</bias_mean>
+                <bias_stddev>0.0000008</bias_stddev>
+                </noise>
+            </x>
+            <y>
+                <noise type="gaussian">
+                <mean>0.0</mean>
+                <stddev>2e-4</stddev>
+                <bias_mean>0.0000075</bias_mean>
+                <bias_stddev>0.0000008</bias_stddev>
+                </noise>
+            </y>
+            <z>
+                <noise type="gaussian">
+                <mean>0.0</mean>
+                <stddev>2e-4</stddev>
+                <bias_mean>0.0000075</bias_mean>
+                <bias_stddev>0.0000008</bias_stddev>
+                </noise>
+            </z>
+            </angular_velocity>
+            <linear_acceleration>
+            <x>
+                <noise type="gaussian">
+                <mean>0.0</mean>
+                <stddev>1.7e-2</stddev>
+                <bias_mean>0.1</bias_mean>
+                <bias_stddev>0.001</bias_stddev>
+                </noise>
+            </x>
+            <y>
+                <noise type="gaussian">
+                <mean>0.0</mean>
+                <stddev>1.7e-2</stddev>
+                <bias_mean>0.1</bias_mean>
+                <bias_stddev>0.001</bias_stddev>
+                </noise>
+            </y>
+            <z>
+                <noise type="gaussian">
+                <mean>0.0</mean>
+                <stddev>1.7e-2</stddev>
+                <bias_mean>0.1</bias_mean>
+                <bias_stddev>0.001</bias_stddev>
+                </noise>
+            </z>
+            </linear_acceleration>
+        </imu>
+        </sensor>
+    </gazebo>
     <gazebo>
         <plugin name='gz::sim::systems::MulticopterMotorModel' filename='ignition-gazebo-multicopter-motor-model-system'>
@@ -290,69 +381,11 @@
             </rotorConfiguration>
         </plugin>
-        <sensor name="imu_sensor" type="imu">
-            <topic>/model/tello/imu</topic>
-            <frame_id>base_link</frame_id>
-            <ignition_frame_id>base_link</ignition_frame_id>
-            <plugin filename="libignition-gazebo-imu-system.so" name="ignition::gazebo::systems::Imu">
-                <initial_orientation_as_reference>false</initial_orientation_as_reference>
-            </plugin>
-            <always_on>true</always_on>
-            <update_rate>200</update_rate>
-            <visualize>true</visualize>
-            <imu>
-                <angular_velocity>
-                <x>
-                    <noise type="gaussian">
-                    <mean>0.0</mean>
-                    <stddev>2e-4</stddev>
-                    <bias_mean>0.0000075</bias_mean>
-                    <bias_stddev>0.0000008</bias_stddev>
-                    </noise>
-                </x>
-                <y>
-                    <noise type="gaussian">
-                    <mean>0.0</mean>
-                    <stddev>2e-4</stddev>
-                    <bias_mean>0.0000075</bias_mean>
-                    <bias_stddev>0.0000008</bias_stddev>
-                    </noise>
-                </y>
-                <z>
-                    <noise type="gaussian">
-                    <mean>0.0</mean>
-                    <stddev>2e-4</stddev>
-                    <bias_mean>0.0000075</bias_mean>
-                    <bias_stddev>0.0000008</bias_stddev>
-                    </noise>
-                </z>
-                </angular_velocity>
-                <linear_acceleration>
-                <x>
-                    <noise type="gaussian">
-                    <mean>0.0</mean>
-                    <stddev>1.7e-2</stddev>
-                    <bias_mean>0.1</bias_mean>
-                    <bias_stddev>0.001</bias_stddev>
-                    </noise>
-                </x>
-                <y>
-                    <noise type="gaussian">
-                    <mean>0.0</mean>
-                    <stddev>1.7e-2</stddev>
-                    <bias_mean>0.1</bias_mean>
-                    <bias_stddev>0.001</bias_stddev>
-                    </noise>
-                </y>
-                <z>
-                    <noise type="gaussian">
-                    <mean>0.0</mean>
-                    <stddev>1.7e-2</stddev>
-                    <bias_mean>0.1</bias_mean>
-                    <bias_stddev>0.001</bias_stddev>
-                    </noise>
-                </z>
-                </linear_acceleration>
-            </imu>
-        </sensor>
+        <plugin name='ignition::gazebo::systems::OdometryPublisher' filename='ignition-gazebo-odometry-publisher-system'>
+            <dimensions>3</dimensions>
+            <odom_frame>/odom</odom_frame>
+            <odom_topic>tello/odometry</odom_topic>
+            <robot_base_frame>base_link</robot_base_frame>
+            <tf_topic>/tello/tf</tf_topic>
+        </plugin>
     </gazebo>
     <!--

File: src/tello_description/urdf/tello.urdf.xacro (robot description, xacro)
@@ -2,5 +2,5 @@
 <!-- Body coordinates are: x forward, y left, z up; rotation is: roll right, pitch forward, yaw left -->
 <!-- See http://www.ros.org/reps/rep-0103.html -->
-<robot name="tello">
+<robot name="tello" xmlns:xacro="http://ros.org/wiki/xacro">
     <!-- Materials -->
     <material name="gray">
@@ -174,4 +174,95 @@
         <axis xyz="0 0 1"/>
     </joint>
+    <link name="camera_optical_frame"/>
+    <joint name="camera_joint" type="fixed">
+        <origin xyz="0.059 0 0" rpy="0 0 0"/>
+        <parent link="base_link"/>
+        <child link="camera_optical_frame"/>
+    </joint>
+    <gazebo reference="camera_optical_frame">
+        <sensor name="depth_camera" type="depth">
+            <update_rate>10</update_rate>
+            <topic>ircam1</topic>
+            <camera>
+            <horizontal_fov>1.05</horizontal_fov>
+            <image>
+                <width>640</width>
+                <height>480</height>
+                <format>R_FLOAT32</format>
+            </image>
+            <clip>
+                <near>0.1</near>
+                <far>10.0</far>
+            </clip>
+            </camera>
+            <always_on>true</always_on>
+            <visualize>true</visualize>
+        </sensor>
+    </gazebo>
+    <gazebo reference="base_link">
+        <sensor name="imu_sensor" type="imu">
+        <topic>/tello/imu</topic>
+        <plugin filename="gz-sim-imu-system" name="gz::sim::systems::Imu">
+            <initial_orientation_as_reference>false</initial_orientation_as_reference>
+        </plugin>
+        <always_on>true</always_on>
+        <update_rate>200</update_rate>
+        <visualize>true</visualize>
+        <imu>
+            <angular_velocity>
+            <x>
+                <noise type="gaussian">
+                <mean>0.0</mean>
+                <stddev>2e-4</stddev>
+                <bias_mean>0.0000075</bias_mean>
+                <bias_stddev>0.0000008</bias_stddev>
+                </noise>
+            </x>
+            <y>
+                <noise type="gaussian">
+                <mean>0.0</mean>
+                <stddev>2e-4</stddev>
+                <bias_mean>0.0000075</bias_mean>
+                <bias_stddev>0.0000008</bias_stddev>
+                </noise>
+            </y>
+            <z>
+                <noise type="gaussian">
+                <mean>0.0</mean>
+                <stddev>2e-4</stddev>
+                <bias_mean>0.0000075</bias_mean>
+                <bias_stddev>0.0000008</bias_stddev>
+                </noise>
+            </z>
+            </angular_velocity>
+            <linear_acceleration>
+            <x>
+                <noise type="gaussian">
+                <mean>0.0</mean>
+                <stddev>1.7e-2</stddev>
+                <bias_mean>0.1</bias_mean>
+                <bias_stddev>0.001</bias_stddev>
+                </noise>
+            </x>
+            <y>
+                <noise type="gaussian">
+                <mean>0.0</mean>
+                <stddev>1.7e-2</stddev>
+                <bias_mean>0.1</bias_mean>
+                <bias_stddev>0.001</bias_stddev>
+                </noise>
+            </y>
+            <z>
+                <noise type="gaussian">
+                <mean>0.0</mean>
+                <stddev>1.7e-2</stddev>
+                <bias_mean>0.1</bias_mean>
+                <bias_stddev>0.001</bias_stddev>
+                </noise>
+            </z>
+            </linear_acceleration>
+        </imu>
+        </sensor>
+    </gazebo>
     <gazebo>
         <plugin name='gz::sim::systems::MulticopterMotorModel' filename='ignition-gazebo-multicopter-motor-model-system'>
@@ -290,69 +381,11 @@
             </rotorConfiguration>
         </plugin>
-        <sensor name="imu_sensor" type="imu">
-            <topic>/model/tello/imu</topic>
-            <frame_id>base_link</frame_id>
-            <ignition_frame_id>base_link</ignition_frame_id>
-            <plugin filename="libignition-gazebo-imu-system.so" name="ignition::gazebo::systems::Imu">
-                <initial_orientation_as_reference>false</initial_orientation_as_reference>
-            </plugin>
-            <always_on>true</always_on>
-            <update_rate>200</update_rate>
-            <visualize>true</visualize>
-            <imu>
-                <angular_velocity>
-                <x>
-                    <noise type="gaussian">
-                    <mean>0.0</mean>
-                    <stddev>2e-4</stddev>
-                    <bias_mean>0.0000075</bias_mean>
-                    <bias_stddev>0.0000008</bias_stddev>
-                    </noise>
-                </x>
-                <y>
-                    <noise type="gaussian">
-                    <mean>0.0</mean>
-                    <stddev>2e-4</stddev>
-                    <bias_mean>0.0000075</bias_mean>
-                    <bias_stddev>0.0000008</bias_stddev>
-                    </noise>
-                </y>
-                <z>
-                    <noise type="gaussian">
-                    <mean>0.0</mean>
-                    <stddev>2e-4</stddev>
-                    <bias_mean>0.0000075</bias_mean>
-                    <bias_stddev>0.0000008</bias_stddev>
-                    </noise>
-                </z>
-                </angular_velocity>
-                <linear_acceleration>
-                <x>
-                    <noise type="gaussian">
-                    <mean>0.0</mean>
-                    <stddev>1.7e-2</stddev>
-                    <bias_mean>0.1</bias_mean>
-                    <bias_stddev>0.001</bias_stddev>
-                    </noise>
-                </x>
-                <y>
-                    <noise type="gaussian">
-                    <mean>0.0</mean>
-                    <stddev>1.7e-2</stddev>
-                    <bias_mean>0.1</bias_mean>
-                    <bias_stddev>0.001</bias_stddev>
-                    </noise>
-                </y>
-                <z>
-                    <noise type="gaussian">
-                    <mean>0.0</mean>
-                    <stddev>1.7e-2</stddev>
-                    <bias_mean>0.1</bias_mean>
-                    <bias_stddev>0.001</bias_stddev>
-                    </noise>
-                </z>
-                </linear_acceleration>
-            </imu>
-        </sensor>
+        <plugin name='ignition::gazebo::systems::OdometryPublisher' filename='ignition-gazebo-odometry-publisher-system'>
+            <dimensions>3</dimensions>
+            <odom_frame>/odom</odom_frame>
+            <odom_topic>tello/odometry</odom_topic>
+            <robot_base_frame>base_link</robot_base_frame>
+            <tf_topic>/tello/tf</tf_topic>
+        </plugin>
     </gazebo>
     <!--
